File: hardware/lxbmc.kicad_pcb (KiCad board)
At the start: 4 copper layers, 100 x 69.5 mm, 26 parts, among them J1 Conn_02x05_Odd_Even, J2 Screw_Terminal_01x04, J3 0826-1X1T-GH-F, J4 Screw_Terminal_01x03, J5 7790, J6 7790, J7 7790, J8 7790, J9 Screw_Terminal_01x04, U1 RPI4CM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

Commit message: m
Parts:
- removed J2: Screw_Terminal_01x04, TerminalBlock_MetzConnect:TerminalBlock_MetzConnect_Type059_RT06304HBWC_1x04_P3.50mm_Horizontal
- added C4: 100nF, Capacitor_SMD:C_0603_1608Metric, F.Cu at (82.2, 11.1)
- added D3: LED, LED_SMD:LED_0402_1005Metric, F.Cu at (30.5, 7.00)
- added D4: LED, LED_SMD:LED_0402_1005Metric, F.Cu at (33.0, 7.00)
- added D5: LED, LED_SMD:LED_0402_1005Metric, F.Cu at (62.5, 6.50)
- added D6: LED, LED_SMD:LED_0402_1005Metric, F.Cu at (25.5, 7.00)
- added D7: LED, LED_SMD:LED_0402_1005Metric, F.Cu at (62.5, 15.0)
- added D8: LED, LED_SMD:LED_0402_1005Metric, F.Cu at (62.5, 10.5)
- added D9: LED, LED_SMD:LED_0402_1005Metric, F.Cu at (62.5, 19.0)
- added FAN1: Fan_4pin, Connector_Molex:Molex_KK-254_AE-6410-04A_1x04_P2.54mm_Vertical, F.Cu at (92.8, 22.6)
- added FAN2: Fan_4pin, Connector_Molex:Molex_KK-254_AE-6410-04A_1x04_P2.54mm_Vertical, F.Cu at (84.0, 22.6)
- added J10: Conn_01x03_Odd_Even, Connector_PinHeader_2.54mm:PinHeader_1x03_P2.54mm_Vertical, F.Cu at (4.00, 6.00)
- added J11: Conn_01x03, Connector_Molex:Molex_KK-254_AE-6410-03A_1x03_P2.54mm_Vertical, B.Cu at (47.5, 9.50)
- added R10: 470, Resistor_SMD:R_0402_1005Metric, F.Cu at (25.5, 9.00)
- added R11: 1K, Resistor_SMD:R_0402_1005Metric, F.Cu at (60.5, 15.0)
- added R12: 470, Resistor_SMD:R_0402_1005Metric, F.Cu at (60.5, 10.5)
- added R13: 36K 1%, Resistor_SMD:R_0402_1005Metric, F.Cu at (80.8, 2.72)
- added R14: 2K, Resistor_SMD:R_0402_1005Metric, F.Cu at (60.5, 19.0)
- added R15: 4.7K, Resistor_SMD:R_0402_1005Metric, F.Cu at (45.0, 9.00)
- added R7: 470, Resistor_SMD:R_0402_1005Metric, F.Cu at (30.5, 9.00)
- added R8: 470, Resistor_SMD:R_0402_1005Metric, F.Cu at (33.0, 9.00)
- added R9: 1K, Resistor_SMD:R_0402_1005Metric, F.Cu at (60.5, 6.50)
- added U2: EMC2301, Package_SO:MSOP-8_3x3mm_P0.65mm, F.Cu at (81.9, 6.66)
- D1: footprint LED_SMD:LED_0603_1608Metric -> LED_SMD:LED_0402_1005Metric
- J4: value Screw_Terminal_01x03 -> Conn_01x03; footprint TerminalBlock_MetzConnect:TerminalBlock_MetzConnect_Type059_RT06303HBWC_1x03_P3.50mm_Horizontal -> Connector_Molex:Molex_KK-254_AE-6410-03A_1x03_P2.54mm_Vertical
- J9: value Screw_Terminal_01x04 -> PSU; footprint TerminalBlock_MetzConnect:TerminalBlock_MetzConnect_Type059_RT06304HBWC_1x04_P3.50mm_Horizontal -> Connector_Molex:Molex_Mini-Fit_Jr_5566-10A_2x05_P4.20mm_Vertical
- R1, R2, R3, R4, R5: footprint Resistor_SMD:R_0603_1608Metric -> Resistor_SMD:R_0402_1005Metric
- RLA1: footprint aep:G3VM-61G1 -> dg_relay:G3VM-SOP
- U1: footprint aep3:rpiCM4 -> dg_rpi:rpi_cm4
- moved D1 69.1 mm to (28.0, 7.00), turned to 90 degrees
- moved R4 68.4 mm to (28.0, 9.00), turned to 270 degrees
- moved J9 63.6 mm to (75.5, 5.00), turned to 270 degrees
- moved RLA1 12.1 mm to (60.5, 25.8), turned to 180 degrees
- moved R5 10.1 mm to (35.3, 48.4), turned to 270 degrees
- moved R1 3.47 mm to (67.2, 29.5), turned to 270 degrees
- moved J4 3.04 mm to (37.5, 9.50), turned to 0 degrees
- moved C1 2.10 mm to (22.6, 11.4), turned to 0 degrees
- moved R3 1.90 mm to (63.9, 21.2)
- moved C2 1.11 mm to (22.6, 13.7), turned to 0 degrees
- moved USB1 1.00 mm to (26.0, 61.5)
- renumbered J1 to USB1
Connections:
- net Net-(R3-Pad1) renamed RELAY
- J4 pad 1: /TX -> GND
- J4 pad 2: GND -> +5V
- J4 pad 3: /RX -> W1
- J9 pad 1: (no net) -> GND
- J9 pad 2: USB- -> GND
- J9 pad 3: USB+ -> GND
- R1 pad 1: ETH_LEDY -> ETH_LED3
- R2 pad 1: ETH_LEDG -> ETH_LED1
- R4 pad 2: Net-(R4-Pad2) -> ETH_LED1
- U1 pad 15: ETH_LEDG -> ETH_LED3
- U1 pad 17: ETH_LEDY -> ETH_LED2
- U1 pad 19: (no net) -> ETH_LED1
- U1 pad 21: Net-(R4-Pad2) -> LED_ACT
- U1 pad 39: (no net) -> /TX
- U1 pad 40: (no net) -> /RX
- U1 pad 51: /RX -> /DEBUG_RX
- U1 pad 54: (no net) -> W1
- U1 pad 55: /TX -> /DEBUG_TX
- U1 pad 80: (no net) -> /SCL
- U1 pad 82: (no net) -> /SDA
Routing:
- net /SDA: track 0.00 -> 87.0 mm, vias 0 -> 2
- net /SCL: track 0.00 -> 80.9 mm, vias 0 -> 2
- net Net-(R4-Pad2): track 68.4 -> 0.00 mm, vias 2 -> 0
- net ETH_LED1: track 0.00 -> 56.3 mm, vias 0 -> 2
- net ETH_LEDG: track 53.0 -> 0.00 mm, vias 2 -> 0
- net ETH_LED3: track 0.00 -> 50.3 mm
- net +5V: track 54.1 -> 101.5 mm
- net pi3.3: track 133.1 -> 175.3 mm, vias 2 -> 4
- net ETH_LEDY: track 41.6 -> 0.00 mm, vias 2 -> 0
- net +12V: track 0.00 -> 37.7 mm, vias 0 -> 1
- net W1: track 0.00 -> 35.0 mm, vias 0 -> 1
- net /DEBUG_TX: track 0.00 -> 30.6 mm
- net /TX: track 17.9 -> 46.2 mm
- net USB+: track 53.9 -> 26.8 mm
- net USB-: track 53.9 -> 26.8 mm
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Other:
- board text added: "12V"
- board text added: "1WIRE"
- board text added: "5VSB"
- board text added: "ACT"
- board text added: "DEBUG"
- board text added: "ETH1"
- board text added: "ETH2"
- board text added: "ETH3"
- board text added: "PWM"
- board text added: "PWROK"
- board text added: "SENSOR"
- board text added: "SERIAL"
- board text added: "TACH"
- board text added: "USB"
- board text added: "biome.devguard.io lxbmc v2"
- board text removed: "PWOK"
