File: hardware/lxbmc.sch (KiCad schematic (older format))
At the start: 26 parts, among them J1 Conn_02x05_Odd_Even, J2 Screw_Terminal_01x04, J3 0826-1X1T-GH-F, J4 Screw_Terminal_01x03, J5 7790, J6 7790, J7 7790, J8 7790, J9 Screw_Terminal_01x04, U1 RPI4CM, X1 DF40HC_3.0_-100DS-0.4V_51_PNP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, X2 DF40HC_3.0_-100DS-0.4V_51_PNP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

Commit message: m
Parts:
- removed J2, J9: Screw_Terminal_01x04, TerminalBlock_MetzConnect:TerminalBlock_MetzConnect_Type059_RT06304HBWC_1x04_P3.50mm_Horizontal, symbol Connector:Screw_Terminal_01x04
- removed J4: Screw_Terminal_01x03, TerminalBlock_MetzConnect:TerminalBlock_MetzConnect_Type059_RT06303HBWC_1x03_P3.50mm_Horizontal, symbol Connector:Screw_Terminal_01x03
- removed unit 2 of U1
- removed unit 4 of U1
- removed unit 5 of U1
- removed unit 7 of U1
- removed unit 8 of U1
- added C4: 100nF, Capacitor_SMD:C_0603_1608Metric, symbol Device:C
- added D3, D4, D5, D6, D7, D8, D9: LED, LED_SMD:LED_0402_1005Metric, symbol Device:LED
- added FAN1, FAN2: Fan_4pin, Connector_Molex:Molex_KK-254_AE-6410-04A_1x04_P2.54mm_Vertical, symbol Motor:Fan_4pin
- added J10: Conn_01x03_Odd_Even, Connector_PinHeader_2.54mm:PinHeader_1x03_P2.54mm_Vertical, symbol Connector_Generic:Conn_01x03
- added J11, J4: Conn_01x03, Connector_Molex:Molex_KK-254_AE-6410-03A_1x03_P2.54mm_Vertical, symbol Connector_Generic:Conn_01x03
- added J9: PSU, Connector_Molex:Molex_Mini-Fit_Jr_5566-10A_2x05_P4.20mm_Vertical, symbol Connector_Generic:Conn_02x05_Counter_Clockwise
- added R10, R12, R7, R8: 470, Resistor_SMD:R_0402_1005Metric, symbol Device:R
- added R11, R9: 1K, Resistor_SMD:R_0402_1005Metric, symbol Device:R
- added R13: 36K 1%, Resistor_SMD:R_0402_1005Metric, symbol Device:R
- added R14: 2K, Resistor_SMD:R_0402_1005Metric, symbol Device:R
- added R15: 4.7K, Resistor_SMD:R_0402_1005Metric, symbol Device:R
- added U2: EMC2301, Package_SO:MSOP-8_3x3mm_P0.65mm, symbol aep:EMC2301
- C1: JLC# (none) -> C14858
- C2: JLC# (none) -> C15850
- D1: footprint LED_SMD:LED_0603_1608Metric -> LED_SMD:LED_0402_1005Metric; JLC# (none) -> C130723
- R1, R2, R3, R4: footprint Resistor_SMD:R_0603_1608Metric -> Resistor_SMD:R_0402_1005Metric; LCSC# (none) -> C25117
- R5: footprint Resistor_SMD:R_0603_1608Metric -> Resistor_SMD:R_0402_1005Metric
- RLA1: footprint aep:G3VM-61G1 -> dg_relay:G3VM-SOP; symbol aep:G3VM-61G1 -> dg_relay:G3VM-61VY2-TR
- U1: footprint aep3:rpiCM4 -> dg_rpi:rpi_cm4; symbol mikucukyilmaz:RPI4CM -> dg_rpi:rpi_cm4
- renumbered J1 to USB1
Connections:
- net +5V: now also D5.2 (A), J4.2 (Pin_2), J9.6 (Pin_6), R15.1
- net GND: now also C4.2, FAN1.1 (-), FAN2.1 (-), J10.2 (Pin_2), J11.1 (Pin_1), J4.1 (Pin_1), J9.1 (Pin_1), J9.2 (Pin_2), J9.3 (Pin_3), J9.4 (Pin_4), J9.5 (Pin_5), R11.2, R14.2, R9.2, U2.4 (GND)
- net PS_ON: now also J9.7 (Pin_7)
- net PWR_OK: now also D7.2 (A), J9.8 (Pin_8)
- net RX: now also U1.40 (GPIO9), J11.2 (Pin_2); no longer U1.51 (GPIO15/UART_RX)
- net TX: now also U1.39 (GPIO8), J11.3 (Pin_3); no longer U1.55 (GPIO14/UART_TX)
- net pi3.3: now also C4.1, D3.2 (A), D4.2 (A), D6.2 (A), D8.2 (A), R13.2, U2.3 (VDD)
- net ETH_LED1: now reaches R4.2
- net ETH_LED1: now also R2.1, U1.19 (Ethernet_nLED1_(speed,yellow,_3.3V)); no longer U1.21 (Pi_nLED_Activity)
- net SCL: now reaches U1.80 (SCL)
- net SCL: now also U2.2 (SMCLK)
- net SDA: now reaches U1.82 (SDA)
- net SDA: now also U2.1 (SMDATA)
- net RELAY: now reaches R3.1, U1.34 (GPIO5)
- net RELAY: now also R12.2
- net W1: now reaches U1.54 (GPIO4)
- net W1: now also J4.3 (Pin_3), R15.2
- net ETH_LEDG renamed ETH_LED3
- net ETH_LED3: now also R1.1, R8.2; no longer R2.1
- net ETH_LEDY renamed ETH_LED2
- net ETH_LED2: now also R7.2; no longer R1.1
- new net: FAN1.4 (PWM), FAN2.4 (PWM), U2.5 (PWM)
- new net: FAN1.3 (Tacho), R13.1, U2.6 (TACH)
- new net: D9.1 (K), R14.1
- new net: D7.1 (K), R11.1
- new net: D3.1 (K), R7.1
- new net: D4.1 (K), R8.1
- new net: D5.1 (K), R9.1
- new net: D6.1 (K), R10.1
- new net: D8.1 (K), R12.1
- new net +12V: D9.2 (A), FAN1.2 (+), FAN2.2 (+), J9.10 (Pin_10), J9.9 (Pin_9)
- new net DEBUG_RX: J10.3 (Pin_3), U1.51 (GPIO15/UART_RX)
- new net DEBUG_TX: J10.1 (Pin_1), U1.55 (GPIO14/UART_TX)
- new net LED_ACT: R10.2, U1.21 (Pi_nLED_Activity)
- no-connect marks 6 -> 11
Other:
- moved on the sheet: R3, RLA1, USB1
